File: output/_autosave-new.kicad_pcb (KiCad board)
At the start: 2 copper layers, 298.5 x 84.2 mm, 111 parts, among them SW1 SW_PUSH, U1 ATMEGA32U4, X1 XTAL_GND

Commit message: feat: added now support
Parts:
- moved C1 166.2 mm to (164.8, 71.8)
- moved C2 166.2 mm to (174.8, 71.8)
- moved X1 166.2 mm to (169.8, 71.8)
- moved U1 153.6 mm to (189.5, 67.2), turned to 90 degrees
- moved C3 153.4 mm to (180.5, 67.2)
- moved R2 153.4 mm to (200.5, 70.2)
- moved R3 153.4 mm to (180.5, 70.2)
- moved R4 153.4 mm to (180.5, 74.2)
- moved C4 64.8 mm to (267.5, 72.8)
- moved C5 64.8 mm to (272.5, 72.8)
- moved C6 64.8 mm to (277.5, 72.8)
- moved C7 64.8 mm to (282.5, 72.8)
- moved R1 54.4 mm to (287.8, 37.5)
- moved SW1 54.4 mm to (287.8, 32.5)
- moved USB1 2.50 mm to (147.8, 2.00)
Connections:
- net Net-(U1-Pad10) renamed /row2
- net Net-(U1-Pad11) renamed /row3
- net Net-(U1-Pad8) renamed /row0
- net Net-(U1-Pad9) renamed /row1
- U1 pad 12: Net-(U1-Pad12) -> /col3
- U1 pad 18: Net-(U1-Pad18) -> /col12
- U1 pad 19: Net-(U1-Pad19) -> /col13
- U1 pad 20: Net-(U1-Pad20) -> /col14
- U1 pad 28: Net-(U1-Pad28) -> /col0
- U1 pad 29: Net-(U1-Pad29) -> /col1
- U1 pad 30: Net-(U1-Pad30) -> /col2
- U1 pad 31: Net-(U1-Pad31) -> /col10
- U1 pad 32: Net-(U1-Pad32) -> /col11
Other:
- board text removed: "Reset button"
