File: output/new.kicad_pcb (KiCad board)
At the start: 2 copper layers, 298.5 x 84.2 mm, 111 parts, among them SW1 SW_PUSH, U1 ATMEGA32U4, X1 XTAL_GND

Commit message: feat: PCB generation finalized
Parts:
- moved C1 5.00 mm to (300.5, 20.0)
- moved C2 5.00 mm to (310.5, 20.0)
- moved C3 5.00 mm to (300.5, 5.00)
- moved C4 5.00 mm to (300.5, 30.0)
- moved C5 5.00 mm to (305.5, 30.0)
- moved C6 5.00 mm to (310.5, 30.0)
- moved C7 5.00 mm to (315.5, 30.0)
- moved R1 5.00 mm to (309.5, -5.00)
- moved R2 5.00 mm to (320.5, 8.00)
- moved R3 5.00 mm to (300.5, 8.00)
- moved R4 5.00 mm to (300.5, 12.0)
- moved SW1 5.00 mm to (309.5, -10.0)
- moved U1 5.00 mm to (309.5, 5.00)
- moved X1 5.00 mm to (305.5, 20.0)
- moved USB1 2.50 mm to (147.8, 2.00)
Connections:
- net Net-(U1-Pad10) renamed /row2
- net Net-(U1-Pad11) renamed /row3
- net Net-(U1-Pad8) renamed /row0
- net Net-(U1-Pad9) renamed /row1
- U1 pad 12: Net-(U1-Pad12) -> /col3
- U1 pad 18: Net-(U1-Pad18) -> /col12
- U1 pad 19: Net-(U1-Pad19) -> /col13
- U1 pad 20: Net-(U1-Pad20) -> /col14
- U1 pad 28: Net-(U1-Pad28) -> /col0
- U1 pad 29: Net-(U1-Pad29) -> /col1
- U1 pad 30: Net-(U1-Pad30) -> /col2
- U1 pad 31: Net-(U1-Pad31) -> /col10
- U1 pad 32: Net-(U1-Pad32) -> /col11

Commit message: feat: added microcontroller with row/col connections to schematics
Connections:
- U1 pad 18: /col12 -> /col10
- U1 pad 19: /col13 -> /col11
- U1 pad 20: /col14 -> /col12
- U1 pad 21: Net-(U1-Pad21) -> /col13
- U1 pad 25: Net-(U1-Pad25) -> /col14
- U1 pad 31: /col10 -> /col8
- U1 pad 32: /col11 -> /col9
- U1 pad 38: Net-(U1-Pad38) -> /col7
- U1 pad 39: Net-(U1-Pad39) -> /col6
- U1 pad 40: Net-(U1-Pad40) -> /col5
- U1 pad 41: Net-(U1-Pad41) -> /col4
Routing:
- added copper zone on B.Cu, net GND
- added copper zone on F.Cu, net VCC
- removed copper zone on F.Cu, net GND
- removed copper zone on B.Cu, net VCC
Changed lines of the file:
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@@
   (gr_arc (start 294.5125 80.2) (end 294.5125 80.2) (angle -90) (layer Edge.Cuts) (width 0.2))
   (gr_arc (start -4 80.2) (end -4 80.2) (angle 90) (layer Edge.Cuts) (width 0.2))
-  (zone (net 0) (net_name GND) (layer F.Cu) (hatch edge 0.508)
-    (connect_pads (clearance 0.508))
+  (zone (net 0) (net_name VCC) (layer F.Cu) (hatch edge 0.508)
+    (connect_pads yes (clearance 0.25))
     (min_thickness 0.254)
     (fill yes (arc_segments 16) (thermal_gap 0.508) (thermal_bridge_width 0.508))
@@
     )
   )
-  (zone (net 0) (net_name VCC) (layer B.Cu) (hatch edge 0.508)
-    (connect_pads (clearance 0.508))
+  (zone (net 0) (net_name GND) (layer B.Cu) (hatch edge 0.508)
+    (connect_pads yes (clearance 0.25))
     (min_thickness 0.254)
     (fill yes (arc_segments 16) (thermal_gap 0.508) (thermal_bridge_width 0.508))
@@
       (net 314 "Net-(C2-Pad1)"))
     (pad 18 smd rect (at 0.8 -5.7 270) (size 1.5 0.55) (layers B.Cu B.Paste B.Mask)
+      (net 13 "/col10"))
+    (pad 19 smd rect (at 1.6 -5.7 270) (size 1.5 0.55) (layers B.Cu B.Paste B.Mask)
+      (net 14 "/col11"))
+    (pad 20 smd rect (at 2.4 -5.7 270) (size 1.5 0.55) (layers B.Cu B.Paste B.Mask)
       (net 15 "/col12"))
-    (pad 19 smd rect (at 1.6 -5.7 270) (size 1.5 0.55) (layers B.Cu B.Paste B.Mask)
+    (pad 21 smd rect (at 3.2 -5.7 270) (size 1.5 0.55) (layers B.Cu B.Paste B.Mask)
       (net 16 "/col13"))
-    (pad 20 smd rect (at 2.4 -5.7 270) (size 1.5 0.55) (layers B.Cu B.Paste B.Mask)
-      (net 17 "/col14"))
-    (pad 21 smd rect (at 3.2 -5.7 270) (size 1.5 0.55) (layers B.Cu B.Paste B.Mask)
-      (net 356 "Net-(U1-Pad21)"))
     (pad 22 smd rect (at 4 -5.7 270) (size 1.5 0.55) (layers B.Cu B.Paste B.Mask)
       (net 357 "Net-(U1-Pad22)"))
@@
       (net 2 VCC))
     (pad 25 smd rect (at 5.7 -2.4) (size 1.5 0.55) (layers B.Cu B.Paste B.Mask)
-      (net 360 "Net-(U1-Pad25)"))
+      (net 17 "/col14"))
     (pad 26 smd rect (at 5.7 -1.6) (size 1.5 0.55) (layers B.Cu B.Paste B.Mask)
       (net 361 "Net-(U1-Pad26)"))
@@
       (net 5 "/col2"))
     (pad 31 smd rect (at 5.7 2.4) (size 1.5 0.55) (layers B.Cu B.Paste B.Mask)
-      (net 13 "/col10"))
+      (net 11 "/col8"))
     (pad 32 smd rect (at 5.7 3.2) (size 1.5 0.55) (layers B.Cu B.Paste B.Mask)
-      (net 14 "/col11"))
+      (net 12 "/col9"))
     (pad 33 smd rect (at 5.7 4) (size 1.5 0.55) (layers B.Cu B.Paste B.Mask)
       (net 322 "Net-(R2-Pad1)"))
@@
       (net 372 "Net-(U1-Pad37)"))
     (pad 38 smd rect (at 0.8 5.7 270) (size 1.5 0.55) (layers B.Cu B.Paste B.Mask)
-      (net 373 "Net-(U1-Pad38)"))
+      (net 10 "/col7"))
     (pad 39 smd rect (at 0 5.7 270) (size 1.5 0.55) (layers B.Cu B.Paste B.Mask)
-      (net 374 "Net-(U1-Pad39)"))
+      (net 9 "/col6"))
     (pad 40 smd rect (at -0.8 5.7 270) (size 1.5 0.55) (layers B.Cu B.Paste B.Mask)
-      (net 375 "Net-(U1-Pad40)"))
+      (net 8 "/col5"))
     (pad 41 smd rect (at -1.6 5.7 270) (size 1.5 0.55) (layers B.Cu B.Paste B.Mask)
-      (net 376 "Net-(U1-Pad41)"))
+      (net 7 "/col4"))
     (pad 42 smd rect (at -2.4 5.7 270) (size 1.5 0.55) (layers B.Cu B.Paste B.Mask)
       (net 377 "Net-(U1-Pad42)"))
