File: output/new.sch (KiCad schematic (older format))
At the start: 98 parts

Commit message: feat: schematics row wiring
Parts:
- removed D_ALT (x2), D_M1, D_OPT (x2), D_SHIFT (x2): D, keyboard_parts:D_SOD123_axial, symbol Device:D
- removed K_ALT (x2), K_SHIFT: KEYSW, MX_Alps_Hybrid:MX-1.25U-NoLED, symbol keyboard_parts:KEYSW
- removed K_M1, K_OPT (x2): KEYSW, MX_Alps_Hybrid:MX-1U-NoLED, symbol keyboard_parts:KEYSW
- removed K_SHIFT: KEYSW, MX_Alps_Hybrid:MX-1.75U-NoLED, symbol keyboard_parts:KEYSW
- added D_ALT (x2), D_OPT (x2), D_SHIFT (x2): D, keyboard_parts:D_SOD123_axial, symbol Device:D
- added K_ALT (x2), K_SHIFT: KEYSW, MX_Alps_Hybrid:MX-1.25U-NoLED, symbol keyboard_parts:KEYSW
- added K_OPT (x2): KEYSW, MX_Alps_Hybrid:MX-1U-NoLED, symbol keyboard_parts:KEYSW
- added K_SHIFT: KEYSW, MX_Alps_Hybrid:MX-1.75U-NoLED, symbol keyboard_parts:KEYSW
Connections:
- net labels removed: col0, col1, col10, col11, col12, col13, col14, col2, col3, col4, col5, col6, col7, col8, col9
- wire segments 196 -> 104

Commit message: chore: removed output folder
Parts:
- removed D_ALT (x2), D_OPT (x2), D_SHIFT (x2): D, keyboard_parts:D_SOD123_axial, symbol Device:D
- removed K_ALT (x2), K_SHIFT: KEYSW, MX_Alps_Hybrid:MX-1.25U-NoLED, symbol keyboard_parts:KEYSW
- removed K_OPT (x2): KEYSW, MX_Alps_Hybrid:MX-1U-NoLED, symbol keyboard_parts:KEYSW
- removed K_SHIFT: KEYSW, MX_Alps_Hybrid:MX-1.75U-NoLED, symbol keyboard_parts:KEYSW
- added D_ALT (x2), D_OPT (x2), D_SHIFT (x2): D, keyboard_parts:D_SOD123_axial, symbol Device:D
- added K_ALT (x2), K_SHIFT: KEYSW, MX_Alps_Hybrid:MX-1.25U-NoLED, symbol keyboard_parts:KEYSW
- added K_OPT (x2): KEYSW, MX_Alps_Hybrid:MX-1U-NoLED, symbol keyboard_parts:KEYSW
- added K_SHIFT: KEYSW, MX_Alps_Hybrid:MX-1.75U-NoLED, symbol keyboard_parts:KEYSW
Connections:
- net labels added: col0, col1, col10, col11, col12, col13, col14, col2, col3, col4, col5, col6, col7, col8, col9
- wire segments 104 -> 134

Commit message: feat: initial PCB generator
Parts:
- removed D_ALT (x2), D_CAPS_LOCK, D_OPT (x2), D_SHIFT (x2): D, keyboard_parts:D_SOD123_axial, symbol Device:D
- removed K_ALT (x2), K_CAPS_LOCK, K_SHIFT: KEYSW, MX_Alps_Hybrid:MX-1.25U-NoLED, symbol keyboard_parts:KEYSW
- removed K_OPT (x2): KEYSW, MX_Alps_Hybrid:MX-1U-NoLED, symbol keyboard_parts:KEYSW
- removed K_SHIFT: KEYSW, MX_Alps_Hybrid:MX-1.75U-NoLED, symbol keyboard_parts:KEYSW
- added D_ALT, D_ALT1, D_CAPS, D_OPT, D_OPT1, D_SHIFT, D_SHIFT1: D, keyboard_parts:D_SOD123_axial, symbol Device:D
- added K_ALT, K_ALT1, K_CAPS, K_SHIFT1: KEYSW, MX_Alps_Hybrid:MX-1.25U-NoLED, symbol keyboard_parts:KEYSW
- added K_OPT, K_OPT1: KEYSW, MX_Alps_Hybrid:MX-1U-NoLED, symbol keyboard_parts:KEYSW
- added K_SHIFT: KEYSW, MX_Alps_Hybrid:MX-1.75U-NoLED, symbol keyboard_parts:KEYSW

Commit message: feat: PCB keyboard layout
Parts:
- renumbered D_[ to D_CBRAC, D_] to D_OBRAC, K_[ to K_CBRAC, K_] to K_OBRAC
Changed lines of the file:
@@
 	13800 650 13800 1000
 $Comp
-L keyboard_parts:KEYSW K_[
+L keyboard_parts:KEYSW K_CBRAC
 U 1 1 b1
 P 13500 1000
-F 0 "K_[" H 13500 1233 60  0000 C CNN
+F 0 "K_CBRAC" H 13500 1233 60  0000 C CNN
 F 1 "KEYSW" H 13500 900 60  0001 C CNN
 F 2 "MX_Alps_Hybrid:MX-1U-NoLED" H 13500 1000 60  0001 C CNN
@@
 $EndComp
 $Comp
-L Device:D D_[
+L Device:D D_CBRAC
 U 1 1 b0
 P 13150 1250
-F 0 "D_[" V 13196 1171 50  0000 R CNN
+F 0 "D_CBRAC" V 13196 1171 50  0000 R CNN
 F 1 "D" V 13095 1171 50  0000 R CNN
 F 2 "keyboard_parts:D_SOD123_axial" H 13150 1250 50  0001 C CNN
@@
 	14800 650 14800 1000
 $Comp
-L keyboard_parts:KEYSW K_]
+L keyboard_parts:KEYSW K_OBRAC
 U 1 1 c1
 P 14500 1000
-F 0 "K_]" H 14500 1233 60  0000 C CNN
+F 0 "K_OBRAC" H 14500 1233 60  0000 C CNN
 F 1 "KEYSW" H 14500 900 60  0001 C CNN
 F 2 "MX_Alps_Hybrid:MX-1U-NoLED" H 14500 1000 60  0001 C CNN
@@
 $EndComp
 $Comp
-L Device:D D_]
+L Device:D D_OBRAC
 U 1 1 c0
 P 14150 1250
-F 0 "D_]" V 14196 1171 50  0000 R CNN
+F 0 "D_OBRAC" V 14196 1171 50  0000 R CNN
 F 1 "D" V 14095 1171 50  0000 R CNN
 F 2 "keyboard_parts:D_SOD123_axial" H 14150 1250 50  0001 C CNN

Commit message: feat: added microcontroller with row/col connections to schematics
Parts:
- added U1: ATMEGA32U4, Package_QFP:TQFP-44_10x10mm_P0.8mm, symbol keyboard_parts:ATMEGA32U4
Connections:
- no-connect marks 0 -> 2
Changed lines of the file:
@@
 Comment4 ""
 $EndDescr
+$Comp
+L keyboard_parts:ATMEGA32U4 U1
+U 1 1 21A1
+P 8550 8000
+F 0 "U1" H 8575 9337 60  0000 C CNN
+F 1 "ATMEGA32U4" H 8575 9231 60  0000 C CNN
+F 2 "Package_QFP:TQFP-44_10x10mm_P0.8mm" H 8550 8000 60  0001 C CNN
+F 3 "" H 8550 8000 60  0000 C CNN
+	1    8550 8000
+	1    0    0    -1
+$EndComp
+Text GLabel 7500 7650 0    50   Input ~ 0
+row0
+Text GLabel 7500 7750 0    50   Input ~ 0
+row1
+Text GLabel 7500 7850 0    50   Input ~ 0
+row2
+Text GLabel 7500 7950 0    50   Input ~ 0
+row3
+Text GLabel 9650 8550 2    50   Input ~ 0
+col0
+Text GLabel 9650 8450 2    50   Input ~ 0
+col1
+Text GLabel 9650 8350 2    50   Input ~ 0
+col2
+Text GLabel 7500 8050 0    50   Input ~ 0
+col3
+Text GLabel 9650 7250 2    50   Input ~ 0
+col4
+Text GLabel 9650 7350 2    50   Input ~ 0
+col5
+Text GLabel 9650 7450 2    50   Input ~ 0
+col6
+Text GLabel 9650 7550 2    50   Input ~ 0
+col7
+Text GLabel 9650 8250 2    50   Input ~ 0
+col8
+Text GLabel 9650 8150 2    50   Input ~ 0
+col9
+Text GLabel 7500 8650 0    50   Input ~ 0
+col10
+Text GLabel 7500 8750 0    50   Input ~ 0
+col11
+Text GLabel 7500 8850 0    50   Input ~ 0
+col12
+Text GLabel 7500 8950 0    50   Input ~ 0
+col13
+Text GLabel 9650 8850 2    50   Input ~ 0
+col14
+NoConn ~ 7500 6950
+NoConn ~ 7500 7550
 Text GLabel 900 1400 0    50   Input ~ 0
 row0

Commit message: feat: added USB and USB connection resistors to schematics
Parts:
- added J1: USB_mini_micro_B, keyboard_parts:USB_miniB_hirose_5S8, symbol keyboard_parts:USB_mini_micro_B
- added R1 (x2): 22, Resistor_SMD:R_0805_2012Metric_Pad1.15x1.40mm_HandSolder, symbol Device:R
Connections:
- no-connect marks 2 -> 1
Changed lines of the file:
@@
 Text GLabel 9650 8850 2    50   Input ~ 0
 col14
+$Comp
+L keyboard_parts:USB_mini_micro_B J1
+U 1 1 14A1
+P 6550 7200
+F 0 "J1" H 6432 7491 60  0000 C CNN
+F 1 "USB_mini_micro_B" H 6400 7400 60  0001 C CNN
+F 2 "keyboard_parts:USB_miniB_hirose_5S8" H 6500 7200 60  0001 C CNN
+F 3 "" H 6500 7200 60  0000 C CNN
+	1    6550 7200
+	1    0    0    -1
+$EndComp
+$Comp
+L Device:R R1
+U 1 1 37B1
+P 7200 7150
+F 0 "R3" V 7200 7100 50  0000 C CNN
+F 1 "22" V 7200 7200 50  0000 C CNN
+F 2 "Resistor_SMD:R_0805_2012Metric_Pad1.15x1.40mm_HandSolder" V 7130 7150 50  0001 C CNN
+F 3 "~" H 7200 7150 50  0001 C CNN
+	1    7200 7150
+	0    1    1    0
+$EndComp
+$Comp
+L Device:R R1
+U 1 1 37B1
+P 7200 7250
+F 0 "R3" V 7200 7200 50  0000 C CNN
+F 1 "22" V 7200 7300 50  0000 C CNN
+F 2 "Resistor_SMD:R_0805_2012Metric_Pad1.15x1.40mm_HandSolder" V 7130 7250 50  0001 C CNN
+F 3 "~" H 7200 7250 50  0001 C CNN
+	1    7200 7250
+	0    1    1    0
+$EndComp
 NoConn ~ 7500 6950
-NoConn ~ 7500 7550
 Text GLabel 900 1400 0    50   Input ~ 0
 row0

Commit message: feat: VCC and microcontroller resistors/caps
Parts:
- removed R1 (x2): 22, Resistor_SMD:R_0805_2012Metric_Pad1.15x1.40mm_HandSolder, symbol Device:R
- added C8: 1u, Capacitor_SMD:C_0805_2012Metric_Pad1.15x1.40mm_HandSolder, symbol Device:C_Small
- added R3, R4: 22, Resistor_SMD:R_0805_2012Metric_Pad1.15x1.40mm_HandSolder, symbol Device:R
Connections:
- net labels added: VCC
Changed lines of the file:
@@
 $EndComp
 $Comp
-L Device:R R1
+L Device:R R3
 U 1 1 37B1
 P 7200 7150
-F 0 "R3" V 7200 7100 50  0000 C CNN
-F 1 "22" V 7200 7200 50  0000 C CNN
+F 0 "R3" V 7200 7100 39  0000 C CNN
+F 1 "22" V 7200 7200 39  0000 C CNN
 F 2 "Resistor_SMD:R_0805_2012Metric_Pad1.15x1.40mm_HandSolder" V 7130 7150 50  0001 C CNN
 F 3 "~" H 7200 7150 50  0001 C CNN
@@
 $EndComp
 $Comp
-L Device:R R1
+L Device:R R4
 U 1 1 37B1
 P 7200 7250
-F 0 "R3" V 7200 7200 50  0000 C CNN
-F 1 "22" V 7200 7300 50  0000 C CNN
+F 0 "R3" V 7200 7200 39  0000 C CNN
+F 1 "22" V 7200 7300 39  0000 C CNN
 F 2 "Resistor_SMD:R_0805_2012Metric_Pad1.15x1.40mm_HandSolder" V 7130 7250 50  0001 C CNN
 F 3 "~" H 7200 7250 50  0001 C CNN
@@
 	0    1    1    0
 $EndComp
+$Comp
+L Device:C_Small C8
+U 1 1 1341
+P 7300 7450
+F 0 "C8" V 7350 7550 50  0000 C CNN
+F 1 "1u" V 7350 7350 50  0000 C CNN
+F 2 "Capacitor_SMD:C_0805_2012Metric_Pad1.15x1.40mm_HandSolder" H 7300 7450 50  0001 C CNN
+F 3 "~" H 7300 7450 50  0001 C CNN
+	1    7300 7450
+	0    1    1    0
+$EndComp
+$Comp
+L power:VCC #PWR0101
+U 1 1 13C1
+P 6850 6850
+F 0 "#PWR0107" H 6850 6700 50  0001 C CNN
+F 1 "VCC" H 6867 7023 50  0000 C CNN
+F 2 "" H 6850 6850 50  0001 C CNN
+F 3 "" H 6850 6850 50  0001 C CNN
+	1    6850 6850
+	1    0    0    -1
+$EndComp
 NoConn ~ 7500 6950
